File: pico-devboard/pico-devboard.kicad_sch (KiCad schematic)
At the start: 10 parts, among them J1 Power Header, J2 GPIO Header, J3 Off-board Header, J4 Pico Dev, J5 Pico Dev Programming, SW1 SW_Push_Dual, SW2 SW_SPDT, U1 Pico

Commit message: Silkscreen, small adjustments, readme updates
Parts:
- added J6: Test Header, Connector_PinHeader_2.54mm:PinHeader_1x04_P2.54mm_Vertical, symbol Connector_Generic:Conn_01x04
Connections:
- net +3V3: now also J6.3 (Pin_3)
- net +5V: now also SW2.2 (B), U1.39 (VSYS), U1.40 (VBUS), J6.1 (Pin_1); no longer D1.2 (A), J1.1 (Pin_1), J4.39 (Pin_39), SW2.1 (A)
- net GND: now also J6.4 (Pin_4)
- new net 5V_switched: D1.2 (A), J1.1 (Pin_1), J4.39 (Pin_39), J6.2 (Pin_2), SW2.1 (A)
Other:
- note added: "Connectors from Pico to bread board"
- note added: "Connectors to off-board parts and testing."
- note added: "Zif Socket"
- moved on the sheet: J1, J2

Commit message: Fixing header spacing issue and re-routing
Parts:
- J1, J5: footprint Connector_PinHeader_1.27mm:PinHeader_1x03_P1.27mm_Vertical -> Connector_PinHeader_2.54mm:PinHeader_1x03_P2.54mm_Vertical
- J2: footprint Connector_PinHeader_1.27mm:PinHeader_1x26_P1.27mm_Vertical -> Connector_PinHeader_2.54mm:PinHeader_1x26_P2.54mm_Vertical
- J3: footprint Connector_PinHeader_1.27mm:PinHeader_2x10_P1.27mm_Vertical -> Connector_PinHeader_2.54mm:PinHeader_2x10_P2.54mm_Vertical
Connections:
- net +5V: no longer U1.40 (VBUS)
- net GND: no longer SW2.3 (C)
- no-connect marks 31 -> 33
Other:
- title: (none) -> Pico Dev Board
- moved on the sheet: R1
Changed lines of the file:
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@@
 (kicad_sch (version 20211123) (generator eeschema)
   (paper "A4")
+  (title_block
+    (title "Pico Dev Board")
+    (date "2023-03-07")
+    (rev "A")
+  )
   (junction (at 116.84 41.91) (diameter 0) (color 0 0 0 0)
   )
@@
   (junction (at 134.62 54.61) (diameter 0) (color 0 0 0 0)
   )
-  (junction (at 69.85 26.67) (diameter 0) (color 0 0 0 0)
-  )
   (junction (at 67.31 54.61) (diameter 0) (color 0 0 0 0)
   )
-  (junction (at 67.31 24.13) (diameter 0) (color 0 0 0 0)
-  )
-  (junction (at 82.55 31.75) (diameter 0) (color 0 0 0 0)
+  (junction (at 67.31 26.67) (diameter 0) (color 0 0 0 0)
   )
   (no_connect (at 44.45 77.47))
@@
   (no_connect (at 64.77 31.75))
   (no_connect (at 132.08 31.75))
+  (no_connect (at 64.77 24.13))
   (no_connect (at 29.21 52.07))
   (no_connect (at 29.21 49.53))
@@
   (no_connect (at 29.21 57.15))
   (no_connect (at 29.21 72.39))
+  (no_connect (at 81.28 29.21))
   (no_connect (at 29.21 24.13))
   (wire (pts (xy 132.08 67.31) (xy 134.62 67.31))
@@
     (stroke (width 0) (type default) (color 0 0 0 0))
   )
-  (wire (pts (xy 67.31 24.13) (xy 69.85 24.13))
-    (stroke (width 0) (type default) (color 0 0 0 0))
-  )
   (wire (pts (xy 46.99 78.74) (xy 46.99 77.47))
     (stroke (width 0) (type default) (color 0 0 0 0))
@@
     (stroke (width 0) (type default) (color 0 0 0 0))
   )
-  (wire (pts (xy 69.85 26.67) (xy 64.77 26.67))
-    (stroke (width 0) (type default) (color 0 0 0 0))
-  )
   (wire (pts (xy 193.04 27.94) (xy 195.58 27.94))
     (stroke (width 0) (type default) (color 0 0 0 0))
@@
     (stroke (width 0) (type default) (color 0 0 0 0))
   )
+  (wire (pts (xy 67.31 26.67) (xy 71.12 26.67))
+    (stroke (width 0) (type default) (color 0 0 0 0))
+  )
   (wire (pts (xy 104.14 46.99) (xy 119.38 46.99))
     (stroke (width 0) (type default) (color 0 0 0 0))
@@
     (stroke (width 0) (type default) (color 0 0 0 0))
   )
-  (wire (pts (xy 64.77 24.13) (xy 67.31 24.13))
-    (stroke (width 0) (type default) (color 0 0 0 0))
-  )
   (wire (pts (xy 64.77 49.53) (xy 72.39 49.53))
     (stroke (width 0) (type default) (color 0 0 0 0))
@@
     (stroke (width 0) (type default) (color 0 0 0 0))
   )
-  (wire (pts (xy 82.55 31.75) (xy 83.82 31.75))
-    (stroke (width 0) (type default) (color 0 0 0 0))
-  )
   (wire (pts (xy 264.16 52.07) (xy 270.51 52.07))
     (stroke (width 0) (type default) (color 0 0 0 0))
@@
     (stroke (width 0) (type default) (color 0 0 0 0))
   )
-  (wire (pts (xy 82.55 31.75) (xy 82.55 33.02))
-    (stroke (width 0) (type default) (color 0 0 0 0))
-  )
-  (wire (pts (xy 69.85 24.13) (xy 69.85 26.67))
-    (stroke (width 0) (type default) (color 0 0 0 0))
-  )
   (wire (pts (xy 134.62 41.91) (xy 134.62 54.61))
     (stroke (width 0) (type default) (color 0 0 0 0))
@@
     (stroke (width 0) (type default) (color 0 0 0 0))
   )
-  (wire (pts (xy 81.28 29.21) (xy 82.55 29.21))
-    (stroke (width 0) (type default) (color 0 0 0 0))
-  )
   (wire (pts (xy 123.19 101.6) (xy 123.19 110.49))
     (stroke (width 0) (type default) (color 0 0 0 0))
@@
     (stroke (width 0) (type default) (color 0 0 0 0))
   )
-  (wire (pts (xy 69.85 26.67) (xy 71.12 26.67))
+  (wire (pts (xy 64.77 26.67) (xy 67.31 26.67))
     (stroke (width 0) (type default) (color 0 0 0 0))
   )
@@
     (stroke (width 0) (type default) (color 0 0 0 0))
   )
-  (wire (pts (xy 67.31 20.32) (xy 67.31 24.13))
-    (stroke (width 0) (type default) (color 0 0 0 0))
-  )
   (wire (pts (xy 132.08 49.53) (xy 147.32 49.53))
     (stroke (width 0) (type default) (color 0 0 0 0))
@@
     (stroke (width 0) (type default) (color 0 0 0 0))
   )
+  (wire (pts (xy 67.31 20.32) (xy 67.31 26.67))
+    (stroke (width 0) (type default) (color 0 0 0 0))
+  )
   (wire (pts (xy 193.04 80.01) (xy 205.74 80.01))
     (stroke (width 0) (type default) (color 0 0 0 0))
@@
   )
   (wire (pts (xy 104.14 44.45) (xy 119.38 44.45))
-    (stroke (width 0) (type default) (color 0 0 0 0))
-  )
-  (wire (pts (xy 82.55 29.21) (xy 82.55 31.75))
     (stroke (width 0) (type default) (color 0 0 0 0))
   )
@@
     (pin "1")
   )
-  (symbol (lib_id "power:GND") (at 82.55 33.02 0) (unit 1)
-    (in_bom yes) (on_board yes) (fields_autoplaced)
-    (property "Reference" "#PWR05" (id 0) (at 82.55 39.37 0)
-      (effects (font (size 1.27 1.27)) hide)
-    )
-    (property "Value" "GND" (id 1) (at 82.55 38.1 0))
-    (property "Footprint" "" (id 2) (at 82.55 33.02 0)
-      (effects (font (size 1.27 1.27)) hide)
-    )
-    (property "Datasheet" "" (id 3) (at 82.55 33.02 0)
-      (effects (font (size 1.27 1.27)) hide)
-    )
-    (pin "1")
-  )
-  (symbol (lib_id "Device:R") (at 87.63 31.75 90) (unit 1)
+  (symbol (lib_id "power:GND") (at 91.44 39.37 0) (unit 1)
+    (in_bom yes) (on_board yes) (fields_autoplaced)
+    (property "Reference" "#PWR05" (id 0) (at 91.44 45.72 0)
+      (effects (font (size 1.27 1.27)) hide)
+    )
+    (property "Value" "GND" (id 1) (at 91.44 44.45 0))
+    (property "Footprint" "" (id 2) (at 91.44 39.37 0)
+      (effects (font (size 1.27 1.27)) hide)
+    )
+    (property "Datasheet" "" (id 3) (at 91.44 39.37 0)
+      (effects (font (size 1.27 1.27)) hide)
+    )
+    (pin "1")
+  )
+  (symbol (lib_id "Device:R") (at 91.44 35.56 180) (unit 1)
     (in_bom yes) (on_board yes)
-    (property "Reference" "R1" (id 0) (at 88.9 34.29 90))
-    (property "Value" "R" (id 1) (at 88.9 36.83 90)
-      (effects (font (size 1.27 1.27)) hide)
-    )
-    (property "Footprint" "Resistor_THT:R_Axial_DIN0411_L9.9mm_D3.6mm_P15.24mm_Horizontal" (id 2) (at 87.63 33.528 90)
-      (effects (font (size 1.27 1.27)) hide)
-    )
-    (property "Datasheet" "~" (id 3) (at 87.63 31.75 0)
+    (property "Reference" "R1" (id 0) (at 93.98 36.83 0))
+    (property "Value" "R" (id 1) (at 96.52 34.29 90)
+      (effects (font (size 1.27 1.27)) hide)
+    )
+    (property "Footprint" "Resistor_THT:R_Axial_DIN0411_L9.9mm_D3.6mm_P15.24mm_Horizontal" (id 2) (at 93.218 35.56 90)
+      (effects (font (size 1.27 1.27)) hide)
+    )
+    (property "Datasheet" "~" (id 3) (at 91.44 35.56 0)
       (effects (font (size 1.27 1.27)) hide)
     )
@@
     (property "Reference" "J2" (id 0) (at 187.96 39.37 0))
     (property "Value" "GPIO Header" (id 1) (at 184.15 72.39 90))
-    (property "Footprint" "Connector_PinHeader_1.27mm:PinHeader_1x26_P1.27mm_Vertical" (id 2) (at 187.96 72.39 0)
+    (property "Footprint" "Connector_PinHeader_2.54mm:PinHeader_1x26_P2.54mm_Vertical" (id 2) (at 187.96 72.39 0)
       (effects (font (size 1.27 1.27)) hide)
     )
@@
     (property "Reference" "J3" (id 0) (at 257.81 43.18 0))
     (property "Value" "Off-board Header" (id 1) (at 257.81 45.72 0))
-    (property "Footprint" "Connector_PinHeader_1.27mm:PinHeader_2x10_P1.27mm_Vertical" (id 2) (at 256.54 59.69 0)
+    (property "Footprint" "Connector_PinHeader_2.54mm:PinHeader_2x10_P2.54mm_Vertical" (id 2) (at 256.54 59.69 0)
       (effects (font (size 1.27 1.27)) hide)
     )
@@
     (property "Reference" "J5" (id 0) (at 132.08 96.52 90))
     (property "Value" "Pico Dev Programming" (id 1) (at 125.73 92.71 90))
-    (property "Footprint" "Connector_PinHeader_1.27mm:PinHeader_1x03_P1.27mm_Vertical" (id 2) (at 125.73 96.52 0)
+    (property "Footprint" "Connector_PinHeader_2.54mm:PinHeader_1x03_P2.54mm_Vertical" (id 2) (at 125.73 96.52 0)
       (effects (font (size 1.27 1.27)) hide)
     )
@@
     (property "Reference" "J1" (id 0) (at 187.96 20.32 0))
     (property "Value" "Power Header" (id 1) (at 184.15 25.4 90))
-    (property "Footprint" "Connector_PinHeader_1.27mm:PinHeader_1x03_P1.27mm_Vertical" (id 2) (at 187.96 25.4 0)
+    (property "Footprint" "Connector_PinHeader_2.54mm:PinHeader_1x03_P2.54mm_Vertical" (id 2) (at 187.96 25.4 0)
       (effects (font (size 1.27 1.27)) hide)
     )
@@
     )
     (path "/fd85af7a-aa14-438c-a57a-8d4532c87733"
-      (reference "J1") (unit 1) (value "Power Header") (footprint "Connector_PinHeader_1.27mm:PinHeader_1x03_P1.27mm_Vertical")
+      (reference "J1") (unit 1) (value "Power Header") (footprint "Connector_PinHeader_2.54mm:PinHeader_1x03_P2.54mm_Vertical")
     )
     (path "/6b9d486e-ca76-4de5-9a7b-9c843b661585"
-      (reference "J2") (unit 1) (value "GPIO Header") (footprint "Connector_PinHeader_1.27mm:PinHeader_1x26_P1.27mm_Vertical")
+      (reference "J2") (unit 1) (value "GPIO Header") (footprint "Connector_PinHeader_2.54mm:PinHeader_1x26_P2.54mm_Vertical")
     )
     (path "/9e5935d7-9e8a-4071-a3a7-ffa3f0824557"
-      (reference "J3") (unit 1) (value "Off-board Header") (footprint "Connector_PinHeader_1.27mm:PinHeader_2x10_P1.27mm_Vertical")
+      (reference "J3") (unit 1) (value "Off-board Header") (footprint "Connector_PinHeader_2.54mm:PinHeader_2x10_P2.54mm_Vertical")
     )
     (path "/a2a78647-e546-420c-8669-1d0c87b6e943"
@@
     )
     (path "/d5a8e7a9-bb14-41a4-b1dd-942972499bfa"
-      (reference "J5") (unit 1) (value "Pico Dev Programming") (footprint "Connector_PinHeader_1.27mm:PinHeader_1x03_P1.27mm_Vertical")
+      (reference "J5") (unit 1) (value "Pico Dev Programming") (footprint "Connector_PinHeader_2.54mm:PinHeader_1x03_P2.54mm_Vertical")
     )
     (path "/225111bb-ea7d-4999-951b-36aa6d8b191b"
